Commit message: Changed sphere to cylinder in wheel

File: urdf/modelo_basico_rycsv.urdf (robot description, URDF)
Before this commit: robot robot_rycsv, 7 links, 6 joints
Links:
- link wheel_motor: geometry collision cylinder length=0.05 radius=0.05; visual cylinder length=0.05 radius=0.05

Commit message: Changed radius of cylinder

File: urdf/modelo_basico_rycsv.urdf (robot description, URDF)
Before this commit: robot robot_rycsv, 7 links, 6 joints
Links:
- link wheel_motor: geometry collision cylinder length=0.05 radius=0.055; visual cylinder length=0.05 radius=0.05
